Commit message: feat: change robot wheels to spheres

File: assets/vss_robot.urdf (robot description, URDF)
Before this commit: robot vss, 3 links, 2 joints
Links:
- removed link left_wheel
- removed link right_wheel
- removed link robot_body
- added link body, mass 0.150; collision box size=0.08 0.08 0.054; visual box size=0.08 0.08 0.054
- added link leftWheel, mass 0.015; collision sphere radius=0.026; visual cylinder length=0.0025 radius=0.026
- added link rightWheel, mass 0.015; collision sphere radius=0.026; visual cylinder length=0.0025 radius=0.026
Joints:
- removed joint left_wheel_joint
- removed joint right_wheel_joint
- added joint body_leftWheel: type continuous, parent body, child leftWheel, origin xyz=0.0 0.03875 -0.002 rpy=-1.570796 0.0 0.0, axis 0.0 0.0 1.0, limit effort=0.075 velocity=68.0
- added joint body_rightWheel: type continuous, parent body, child rightWheel, origin xyz=0.0 -0.03875 -0.002 rpy=-1.570796 0.0 0.0, axis 0.0 0.0 1.0, limit effort=0.075 velocity=68.0

Commit message: feat: new robot test parameters

File: assets/vss_robot.urdf (robot description, URDF)
Before this commit: robot vss, 3 links, 2 joints
Links:
- link body: mass 0.150 -> 0.330; geometry collision box size=0.07 0.07 0.042; visual box size=0.07 0.07 0.042
- link leftWheel: mass 0.015 -> 0.02; geometry collision sphere radius=0.024; visual cylinder length=0.0025 radius=0.024
- link rightWheel: mass 0.015 -> 0.02; geometry collision sphere radius=0.024; visual cylinder length=0.0025 radius=0.024
Joints:
- joint body_leftWheel: limit effort=0.075 velocity=68.0 -> effort=0.1 velocity=150.0; origin xyz=0.0 0.03875 -0.002 rpy=-1.570796 0.0 0.0 -> xyz=0.0 0.03375 0.002 rpy=-1.570796 0.0 0.0
- joint body_rightWheel: limit effort=0.075 velocity=68.0 -> effort=0.1 velocity=150.0; origin xyz=0.0 -0.03875 -0.002 rpy=-1.570796 0.0 0.0 -> xyz=0.0 -0.03375 0.002 rpy=-1.570796 0.0 0.0

Commit message: feat: add robots id and team tags

File: assets/vss_robot.urdf (robot description, URDF)
Before this commit: robot vss, 3 links, 2 joints
Links:
- added link tagId; visual box size=0.03 0.05 0.001
- added link tagTeam; visual box size=0.03 0.05 0.001
- link body: geometry collision box size=0.07 0.07 0.042; visual box size=0.07 0.06 0.042
Joints:
- added joint body_tagId: type fixed, parent body, child tagId, origin xyz=0.0175 0.0 0.021
- added joint body_tagTeam: type fixed, parent body, child tagTeam, origin xyz=-0.0175 0.0 0.021
